Commit message: more robot model fixes

File: robot_model/mpo_500/xacros/micro_scan.xacro (robot description, xacro)
@@ -17,5 +17,5 @@
     <origin xyz="-0.0 0 -0.06" rpy="1.57 0 0" />
       <geometry>
-        <mesh filename="package://neo_mpo_500/robot_model/meshes/SICK-MICROSCAN3.dae" scale="0.001 0.001 0.001" />
+        <mesh filename="package://neo_mpo_500/robot_model/mpo_500/meshes/SICK-MICROSCAN3.dae" scale="0.001 0.001 0.001" />
       </geometry>
     </visual>
@@ -23,5 +23,5 @@
     <origin xyz="-0.0 0 -0.06" rpy="1.57 0 0" />
         <geometry>
-          <mesh filename="package://neo_mpo_500/robot_model/meshes/SICK-MICROSCAN3.dae" scale="0.001 0.001 0.001" />
+          <mesh filename="package://neo_mpo_500/robot_model/mpo_500/meshes/SICK-MICROSCAN3.dae" scale="0.001 0.001 0.001" />
           </geometry>
         </collision>

File: robot_model/mpo_500/xacros/mpo_500_body.xacro (robot description, xacro)
@@ -13,5 +13,5 @@
         <origin xyz="0. 0. 0" rpy="-1.571 0 1.571" />
         <geometry>
-            <mesh filename="package://neo_mpo_500/robot_model/meshes/MPO-500-BODY.dae" scale="0.001 0.001 0.001"/>
+            <mesh filename="package://neo_mpo_500/robot_model/mpo_500/meshes/MPO-500-BODY.dae" scale="0.001 0.001 0.001"/>
         </geometry>
       </visual>
@@ -20,5 +20,5 @@
         <geometry>
           <!--<box size="0.68 0.41 0.25"/> -->
-           <mesh filename="package://neo_mpo_500/robot_model/meshes/MPO-500-BODY.dae" scale="0.001 0.001 0.001"/>
+           <mesh filename="package://neo_mpo_500/robot_model/mpo_500/meshes/MPO-500-BODY.dae" scale="0.001 0.001 0.001"/>
         </geometry>
       </collision>

File: robot_model/mpo_500/xacros/omni_wheel.xacro (robot description, xacro)
@@ -20,5 +20,5 @@
      <origin xyz="0 0 0" rpy="0 0 0"/>
      <geometry>
-        <mesh filename="package://neo_mpo_500/robot_model/meshes/MPO-500-WHEEL.dae" scale="0.001 0.001 0.001"/>
+        <mesh filename="package://neo_mpo_500/robot_model/mpo_500/meshes/MPO-500-WHEEL.dae" scale="0.001 0.001 0.001"/>
      </geometry>
     </visual>
@@ -26,5 +26,5 @@
      <origin xyz="0 0 0" rpy="0 0 0" />
      <geometry>
-        <mesh filename="package://neo_mpo_500/robot_model/meshes/MPO-500-WHEEL.dae" scale="0.001 0.001 0.001"/>
+        <mesh filename="package://neo_mpo_500/robot_model/mpo_500/meshes/MPO-500-WHEEL.dae" scale="0.001 0.001 0.001"/>
      </geometry>
     </collision>

File: robot_model/mpo_500/xacros/sick_S300.xacro (robot description, xacro)
@@ -17,5 +17,5 @@
         <origin xyz="0 0 -0.12" rpy="-1.57 0 3.14" />
         <geometry>
-        <mesh filename="package://neo_mpo_500/robot_model/meshes/SICK-S300.dae" scale="0.001 0.001 0.001" />
+        <mesh filename="package://neo_mpo_500/robot_model/mpo_500/meshes/SICK-S300.dae" scale="0.001 0.001 0.001" />
         </geometry>
       </visual>
@@ -23,5 +23,5 @@
         <origin xyz="0 0 -0.12" rpy="-1.57 0 3.14" />
         <geometry>
-        <mesh filename="package://neo_mpo_500/robot_model/meshes/SICK-S300.dae" scale="0.001 0.001 0.001" />
+        <mesh filename="package://neo_mpo_500/robot_model/mpo_500/meshes/SICK-S300.dae" scale="0.001 0.001 0.001" />
         </geometry>
       </collision>

File: robot_model/mpo_500/xacros/sick_laser.xacro (robot description, xacro)
@@ -18,5 +18,5 @@
       <origin xyz="0 0 -0.12" rpy="-1.57 0 3.14" />
         <geometry>
-        <mesh filename="package://neo_mpo_500/robot_model/meshes/SICK-S300.dae" scale="0.001 0.001 0.001" />
+        <mesh filename="package://neo_mpo_500/robot_model/mpo_500/meshes/SICK-S300.dae" scale="0.001 0.001 0.001" />
         </geometry>
       </visual>
@@ -24,5 +24,5 @@
         <origin xyz="0 0 0" rpy="-1.57 0 3.14" />
         <geometry>
-        <mesh filename="package://neo_mpo_500/robot_model/meshes/SICK-S300.dae" scale="0.001 0.001 0.001" />
+        <mesh filename="package://neo_mpo_500/robot_model/mpo_500/meshes/SICK-S300.dae" scale="0.001 0.001 0.001" />
         </geometry>
       </collision>
@@ -30,5 +30,5 @@
 <!--  <origin xyz="-0.0 0 -0.06" rpy="1.57 0 0" />
       <geometry>
-      <mesh filename="package://neo_mpo_500/robot_model/meshes/SICK-MICROSCAN3.dae" scale="0.001 0.001 0.001" />
+      <mesh filename="package://neo_mpo_500/robot_model/mpo_500/meshes/SICK-MICROSCAN3.dae" scale="0.001 0.001 0.001" />
       </geometry>
       </visual>
@@ -36,5 +36,5 @@
  <origin xyz="-0.0 0 -0.06" rpy="1.57 0 0" />
       <geometry>
-        <mesh filename="package://neo_mpo_500/robot_model/meshes/SICK-MICROSCAN3.dae" scale="0.001 0.001 0.001" />
+        <mesh filename="package://neo_mpo_500/robot_model/mpo_500/meshes/SICK-MICROSCAN3.dae" scale="0.001 0.001 0.001" />
         </geometry>
       </collision> -->
