Commit message: new robot model + new laser (microscan3) + new structure for laser configs

File: robot_model/mpo_500/mpo_500.urdf.xacro (robot description, xacro)
@@ -1,8 +1,4 @@
 <?xml version="1.0" ?>
 <robot name="mpo_500" xmlns:xacro="http://www.ros.org/wiki/xacro">
-  <!--GAZEBO REFERENCES -->
-  <xacro:include filename="$(find neo_mpo_500)/robot_model/mpo_500/xacros/mpo_500_gazebo.xacro" />
-  <!-- MATERIALS -->
-  <xacro:include filename="$(find neo_mpo_500)/robot_model/mpo_500/xacros/mpo_500_materials.xacro" />
   <!-- BODY -->
   <xacro:include filename="$(find neo_mpo_500)/robot_model/mpo_500/xacros/mpo_500_body.xacro" />
@@ -10,27 +6,27 @@
   <xacro:include filename="$(find neo_mpo_500)/robot_model/mpo_500/xacros/omni_wheel.xacro" />
   <!-- SENSORS -->
-  <xacro:include filename="$(find neo_mpo_500)/robot_model/mpo_500/xacros/sick_s300_laser.xacro" />
+  <xacro:include filename="$(find neo_mpo_500)/robot_model/mpo_500/xacros/sick_laser.xacro" />
   <!-- Base Macro-->
   <xacro:mpo_500_base name="base_link">
   </xacro:mpo_500_base>
   <!-- Wheel Macro -->
-  <xacro:omni_wheel_250 name="wheel_front_left" parent="base_link" suffix="links">
+  <xacro:omni_wheel_250 name="wheel_front_left" parent="base_link">
   	<origin xyz="0.25 0.28 0.13" rpy="0 0 0" />
   </xacro:omni_wheel_250>
-  <xacro:omni_wheel_250 name="wheel_front_right" parent="base_link" suffix="rechts">
+  <xacro:omni_wheel_250 name="wheel_front_right" parent="base_link">
   	<origin xyz="0.25 -0.28 0.13" rpy="0 0 0" />
   </xacro:omni_wheel_250>
-  <xacro:omni_wheel_250 name="wheel_back_left" parent="base_link" suffix="links">
+  <xacro:omni_wheel_250 name="wheel_back_left" parent="base_link">
   	<origin xyz="-0.25 0.28 0.13" rpy="0 0 0" />
   </xacro:omni_wheel_250>
-  <xacro:omni_wheel_250 name="wheel_back_right" parent="base_link" suffix="rechts">
+  <xacro:omni_wheel_250 name="wheel_back_right" parent="base_link">
   	<origin xyz="-0.25 -0.28 0.13" rpy="0 0 0" />
   </xacro:omni_wheel_250>
   <!-- Sensors -->
-  <xacro:sick_s300_laser_v0 name="sick_s300_laser_front" parent="base_link" ros_topic="sick_s300_front/scan">
-  	<origin xyz="0.442 0 0.420" rpy="0 0 0" />
-  </xacro:sick_s300_laser_v0>
-  <xacro:sick_s300_laser_v0 name="sick_s300_laser_back" parent="base_link" ros_topic="sick_s300_back/scan">
-  	<origin xyz="-0.442 0 0.420" rpy="0 0 3.14" />
-  </xacro:sick_s300_laser_v0>
+  <xacro:sick_laser_v0 name="sick_laser_front" parent="base_link" ros_topic="sick_front/scan">
+  	<origin xyz="0.442 0 0.372" rpy="0 0 0" />
+  </xacro:sick_laser_v0>
+  <xacro:sick_laser_v0 name="sick_laser_back" parent="base_link" ros_topic="sick_back/scan">
+  	<origin xyz="-0.442 0 0.372" rpy="0 0 3.14" />
+  </xacro:sick_laser_v0>
 </robot>

File: robot_model/mpo_500/xacros/mpo_500_body.xacro (robot description, xacro)
@@ -11,15 +11,14 @@
       </inertial>
       <visual>
-        <origin xyz="0. 0. 0.215" rpy="0 0 1.571" />
+        <origin xyz="0. 0. 0" rpy="-1.571 0 1.571" />
         <geometry>
-            <mesh filename="package://neo_mpo_500/robot_model/mpo_500/meshes/MPO-500-BODY.STL"/>
+            <mesh filename="package://neo_mpo_500/robot_model/mpo_500/meshes/MPO-500-BODY.dae" scale="0.001 0.001 0.001"/>
         </geometry>
-        <material name="Neobotix/Grey" />
       </visual>
       <collision>
-        <origin xyz="0. 0. 0.2" rpy="0 0 0" />
+        <origin xyz="0. 0. 0.0" rpy="-1.571 0 1.571" />
         <geometry>
           <!--<box size="0.68 0.41 0.25"/> -->
-          <box size="0.769 0.51 0.307" />
+           <mesh filename="package://neo_mpo_500/robot_model/mpo_500/meshes/MPO-500-BODY.dae" scale="0.001 0.001 0.001"/>
         </geometry>
       </collision>

File: robot_model/mpo_500/xacros/omni_wheel.xacro (robot description, xacro)
@@ -1,6 +1,6 @@
 <?xml version="1.0"?>
 <robot xmlns:xacro="http://www.ros.org/wiki/xacro" name="mpo_500">
-  <xacro:macro name="omni_wheel_250" params="name parent suffix *origin">
-   <joint name="${name}_joint" type="continuous">
+  <xacro:macro name="omni_wheel_250" params="name parent *origin">
+   <joint name="${name}_joint" type="fixed">
     <insert_block name="origin" />
     <axis xyz="0 1 0" />
@@ -11,19 +11,18 @@
    <link name="${name}_link" type="wheel">
     <inertial>
-      <mass value="0.1" />
+      <mass value="9" />
       <origin xyz="0 0 0" rpy="0 0 0" />
       <inertia ixx="0.00044332" ixy="0" ixz="0" iyy="0.00044332" iyz="0" izz="0.00072" />
     </inertial>
     <visual>
-     <origin xyz="0 0 0" rpy="0 0 1.571" />
+     <origin xyz="0 0 0" rpy="0 0 0"/>
      <geometry>
-        <mesh filename="package://neo_mpo_500/robot_model/mpo_500/meshes/Mecanum-Rad ${suffix}.stl" scale="0.001 0.001 0.001"/>
+        <mesh filename="package://neo_mpo_500/robot_model/mpo_500/meshes/MPO-500-WHEEL.dae" scale="0.001 0.001 0.001"/>
      </geometry>
-     <material name="Neobotix/Black" />
     </visual>
     <collision>
-     <origin xyz="0 0 0" rpy="1.59 0 0" />
+     <origin xyz="0 0 0" rpy="0 0 0" />
      <geometry>
-        <cylinder radius="0.12" length="0.1"/>
+        <mesh filename="package://neo_mpo_500/robot_model/mpo_500/meshes/MPO-500-WHEEL.dae" scale="0.001 0.001 0.001"/>
      </geometry>
     </collision>

Commit message: robot models are updated

File: robot_model/mpo_500/mpo_500.urdf.xacro (robot description, xacro)
@@ -1,4 +1,6 @@
 <?xml version="1.0" ?>
 <robot name="mpo_500" xmlns:xacro="http://www.ros.org/wiki/xacro">
+  <!--GAZEBO REFERENCES -->
+  <xacro:include filename="$(find neo_mpo_500)/robot_model/mpo_500/xacros/mpo_500_gazebo.xacro" />
   <!-- BODY -->
   <xacro:include filename="$(find neo_mpo_500)/robot_model/mpo_500/xacros/mpo_500_body.xacro" />
@@ -6,5 +8,10 @@
   <xacro:include filename="$(find neo_mpo_500)/robot_model/mpo_500/xacros/omni_wheel.xacro" />
   <!-- SENSORS -->
-  <xacro:include filename="$(find neo_mpo_500)/robot_model/mpo_500/xacros/sick_laser.xacro" />
+  <!-- Sick S300 - Comment/Uncomment if required  -->
+  <xacro:include filename="$(find neo_mpo_500)/robot_model/mpo_500/xacros/sick_S300.xacro" />
+  <!-- Microscan - Comment/Uncomment if required -->
+  <!-- <xacro:include filename="$(find neo_mpo_500)/robot_model/mpo_500/xacros/micro_scan.xacro" />
+  <xacro:include filename="$(find neo_mpo_500)/robot_model/mpo_500/xacros/imu.xacro" />
+  <xacro:include filename="$(find neo_mpo_500)/robot_model/mpo_500/xacros/ultrasonic.xacro" />-->
   <!-- Base Macro-->
   <xacro:mpo_500_base name="base_link">
@@ -15,5 +22,5 @@
   </xacro:omni_wheel_250>
   <xacro:omni_wheel_250 name="wheel_front_right" parent="base_link">
-  	<origin xyz="0.25 -0.28 0.13" rpy="0 0 0" />
+  	<origin xyz="0.25 -0.28 0.13" rpy="0 0 3.14" />
   </xacro:omni_wheel_250>
   <xacro:omni_wheel_250 name="wheel_back_left" parent="base_link">
@@ -21,12 +28,88 @@
   </xacro:omni_wheel_250>
   <xacro:omni_wheel_250 name="wheel_back_right" parent="base_link">
-  	<origin xyz="-0.25 -0.28 0.13" rpy="0 0 0" />
+  	<origin xyz="-0.25 -0.28 0.13" rpy="0 0 3.14" />
   </xacro:omni_wheel_250>
   <!-- Sensors -->
-  <xacro:sick_laser_v0 name="lidar_1" parent="base_link" ros_topic="sick_front/scan">
-  	<origin xyz="0.442 0 0.372" rpy="0 0 0" />
+   <xacro:sick_laser_v0 name="lidar_1" parent="base_link" ros_topic="lidar_1/scan_filtered">
+     	<origin xyz="0.442 0 0.372" rpy="0 0 0" />
   </xacro:sick_laser_v0>
-  <xacro:sick_laser_v0 name="lidar_2" parent="base_link" ros_topic="sick_back/scan">
-  	<origin xyz="-0.442 0 0.372" rpy="0 0 3.14" />
+   <xacro:sick_laser_v0 name="lidar_2" parent="base_link" ros_topic="lidar_2/scan_filtered">
+     	<origin xyz="-0.442 0 0.372" rpy="0 0 3.14" />
   </xacro:sick_laser_v0>
+       <!--+++++++++++++++++++ IMU ++++++++++++++++++++++++-->
+ <!-- Comment or uncomment based on your requirement -->
+<!--   <xacro:imu name="imu_1" parent="base_link">
+    <origin xyz="0.100 0 0.300" rpy="0 0 3.14" />
+  </xacro:imu> -->
+  <!--+++++++++++++++++++ Ultra Sonic ++++++++++++++++++++++++-->
+  <!-- Comment or uncomment based on your requirement -->
+  <!-- SENSOR 1 -->
+  <!-- xacro:us_sensor name="us_1" parent="base_link">
+    <origin xyz="0.100 0 0.300" rpy="0 3.14 3.14" />
+  </xacro:us_sensor-->
+  <!-- SENSOR 2 -->
+  <!-- xacro:us_sensor name="us_2" parent="base_link">
+    <origin xyz="0.110 0 0.300" rpy="0 3.14 3.14" />
+  </xacro:us_sensor-->
+  <!-- SENSOR 3 -->
+  <!-- xacro:us_sensor name="us_3" parent="base_link">
+    <origin xyz="0.120 0 0.300" rpy="0 3.14 3.14" />
+  </xacro:us_sensor-->
+  <!-- SENSOR 4 -->
+  <!-- xacro:us_sensor name="us_4" parent="base_link">
+    <origin xyz="0.130 0 0.300" rpy="0 3.14 3.14" />
+  </xacro:us_sensor-->
+  <!-- SENSOR 5 -->
+  <!-- xacro:us_sensor name="us_5" parent="base_link">
+    <origin xyz="0.140 0 0.300" rpy="0 3.14 3.14" />
+  </xacro:us_sensor-->
+  <!-- SENSOR 6 -->
+  <!-- xacro:us_sensor name="us_6" parent="base_link">
+    <origin xyz="0.150 0 0.300" rpy="0 3.14 3.14" />
+  </xacro:us_sensor-->
+  <!-- SENSOR 7 -->
+  <!-- xacro:us_sensor name="us_7" parent="base_link">
+    <origin xyz="0.160 0 0.300" rpy="0 3.14 3.14" />
+  </xacro:us_sensor-->
+  <!-- SENSOR 8 -->
+  <!-- xacro:us_sensor name="us_8" parent="base_link">
+    <origin xyz="0.170 0 0.300" rpy="0 3.14 3.14" />
+  </xacro:us_sensor-->
+  <!-- SENSOR 9 -->
+  <!-- xacro:us_sensor name="us_9" parent="base_link">
+    <origin xyz="0.180 0 0.300" rpy="0 3.14 3.14" />
+  </xacro:us_sensor-->
+  <!-- SENSOR 10 -->
+  <!-- xacro:us_sensor name="us_10" parent="base_link">
+    <origin xyz="0.100 0 0.300" rpy="0 3.14 3.14" />
+  </xacro:us_sensor-->
+  <!-- SENSOR 11 -->
+  <!-- xacro:us_sensor name="us_11" parent="base_link">
+    <origin xyz="0.100 0 0.300" rpy="0 3.14 3.14" />
+  </xacro:us_sensor-->
+  <!-- SENSOR 12 -->
+  <!-- xacro:us_sensor name="us_12" parent="base_link">
+    <origin xyz="0.190 0 0.300" rpy="0 3.14 3.14" />
+  </xacro:us_sensor-->
+  <!-- SENSOR 13 -->
+  <!-- xacro:us_sensor name="us_13" parent="base_link">
+    <origin xyz="0.200 0 0.300" rpy="0 3.14 3.14" />
+  </xacro:us_sensor-->
+  <!-- SENSOR 14 -->
+  <!-- xacro:us_sensor name="us_14" parent="base_link">
+    <origin xyz="0.210 0 0.300" rpy="0 3.14 3.14" />
+  </xacro:us_sensor-->
+  <!-- SENSOR 15 -->
+  <!-- xacro:us_sensor name="us_15" parent="base_link">
+    <origin xyz="0.220 0 0.300" rpy="0 3.14 3.14" />
+  </xacro:us_sensor-->
+  <!-- SENSOR 16 -->
+  <!-- xacro:us_sensor name="us_16" parent="base_link">
+    <origin xyz="0.230 0 0.300" rpy="0 3.14 3.14" />
+  </xacro:us_sensor-->
+      <!--Camera  -->
+<!-- <xacro:camera name="camera" parent="base_link">
+    <origin xyz="0 0 0.38" rpy="0 0 0" />
+  </xacro:camera>
+ -->
 </robot>

File: robot_model/mpo_500/xacros/mpo_500_body.xacro (robot description, xacro)
@@ -4,5 +4,5 @@
     <link name="${name}">
       <inertial>
-        <mass value="30" />
+        <mass value="2" />
         <origin xyz="0 0 0" rpy="0 0 0"/>
         <inertia ixx="1.71402" ixy="0.0" ixz="0.0"

File: robot_model/mpo_500/xacros/omni_wheel.xacro (robot description, xacro)
@@ -2,8 +2,10 @@
 <robot xmlns:xacro="http://www.ros.org/wiki/xacro" name="mpo_500">
   <xacro:macro name="omni_wheel_250" params="name parent *origin">
-   <joint name="${name}_joint" type="fixed">
+   <joint name="${name}_joint" type="revolute">
     <insert_block name="origin" />
     <axis xyz="0 1 0" />
-    <joint_properties damping="1" friction="1" />
+    <joint_properties damping="100" friction="1000" />
+        <limit effort="1000.0" lower="-1e+16" upper="1e+16" velocity="3.5"/>
+    <joint_properties damping="1.0" friction="1" />
     <parent link="${parent}" />
     <child link="${name}_link" />
@@ -11,5 +13,5 @@
    <link name="${name}_link" type="wheel">
     <inertial>
-      <mass value="9" />
+      <mass value="1" />
       <origin xyz="0 0 0" rpy="0 0 0" />
       <inertia ixx="0.00044332" ixy="0" ixz="0" iyy="0.00044332" iyz="0" izz="0.00072" />

Commit message: Robot models are updated and depreciation tags are removed

File: robot_model/mpo_500/mpo_500.urdf.xacro (robot description, xacro)
@@ -14,18 +14,20 @@
   <xacro:include filename="$(find neo_mpo_500)/robot_model/mpo_500/xacros/imu.xacro" />
   <xacro:include filename="$(find neo_mpo_500)/robot_model/mpo_500/xacros/ultrasonic.xacro" />
-  <!-- Base Macro-->
-  <xacro:mpo_500_base name="base_link">
+  <link name="base_link" />
+  <!-- Base link macro -->
+  <xacro:mpo_500_base name="base_footprint" parent="base_link">
+    <origin xyz="0 0 0" rpy="0 0 0" />
   </xacro:mpo_500_base>
   <!-- Wheel Macro -->
-  <xacro:omni_wheel_250 name="wheel_front_left" parent="base_link">
+  <xacro:omni_wheel_250 name="wheel_front_left" parent="base_footprint">
   	<origin xyz="0.25 0.28 0.13" rpy="0 0 0" />
   </xacro:omni_wheel_250>
-  <xacro:omni_wheel_250 name="wheel_front_right" parent="base_link">
+  <xacro:omni_wheel_250 name="wheel_front_right" parent="base_footprint">
   	<origin xyz="0.25 -0.28 0.13" rpy="0 0 3.14" />
   </xacro:omni_wheel_250>
-  <xacro:omni_wheel_250 name="wheel_back_left" parent="base_link">
+  <xacro:omni_wheel_250 name="wheel_back_left" parent="base_footprint">
   	<origin xyz="-0.25 0.28 0.13" rpy="0 0 0" />
   </xacro:omni_wheel_250>
-  <xacro:omni_wheel_250 name="wheel_back_right" parent="base_link">
+  <xacro:omni_wheel_250 name="wheel_back_right" parent="base_footprint">
   	<origin xyz="-0.25 -0.28 0.13" rpy="0 0 3.14" />
   </xacro:omni_wheel_250>

File: robot_model/mpo_500/xacros/camera.xacro (robot description, xacro)
@@ -5,5 +5,5 @@
     <joint name="${name}_joint" type="fixed">
       <axis xyz="0 1 0" />
-      <insert_block name="origin" />
+      <xacro:insert_block name="origin" />
       <parent link="${parent}"/>
       <child link="${name}_link"/>

File: robot_model/mpo_500/xacros/imu.xacro (robot description, xacro)
@@ -4,5 +4,5 @@
     <joint name="${name}_joint" type="fixed">
       <axis xyz="0 1 0" />
-      <insert_block name="origin" />
+      <xacro:insert_block name="origin" />
       <parent link="${parent}"/>
       <child link="${name}_link"/>

File: robot_model/mpo_500/xacros/micro_scan.xacro (robot description, xacro)
@@ -4,5 +4,5 @@
     <joint name="${name}_joint" type="fixed">
       <axis xyz="0 1 0" />
-      <insert_block name="origin" />
+      <xacro:insert_block name="origin" />
       <parent link="${parent}"/>
       <child link="${name}_link"/>

File: robot_model/mpo_500/xacros/mpo_500_body.xacro (robot description, xacro)
@@ -1,5 +1,13 @@
 <?xml version="1.0"?>
 <robot xmlns:xacro="http://www.ros.org/wiki/xacro" name="mpo_500">
-  <xacro:macro name="mpo_500_base" params="name">
+  <xacro:macro name="mpo_500_base" params="name parent *origin">
+    <joint name="${name}_joint" type="fixed">
+      <xacro:insert_block name="origin" />
+      <axis xyz="0 0 -1" />
+      <!-- <limit effort="1000.0" lower="-1e+16" upper="1e+16" velocity="3.5"/> -->
+      <joint_properties damping="1" friction="1" />
+      <parent link="${parent}" />
+      <child link="${name}" />
+   </joint>
     <link name="${name}">
       <inertial>

File: robot_model/mpo_500/xacros/omni_wheel.xacro (robot description, xacro)
@@ -3,5 +3,5 @@
   <xacro:macro name="omni_wheel_250" params="name parent *origin">
    <joint name="${name}_joint" type="revolute">
-    <insert_block name="origin" />
+    <xacro:insert_block name="origin" />
     <axis xyz="0 1 0" />
     <joint_properties damping="100" friction="1000" />

File: robot_model/mpo_500/xacros/sick_S300.xacro (robot description, xacro)
@@ -4,5 +4,5 @@
     <joint name="${name}_joint" type="fixed">
       <axis xyz="0 1 0" />
-      <insert_block name="origin" />
+      <xacro:insert_block name="origin" />
       <parent link="${parent}"/>
       <child link="${name}_link"/>

File: robot_model/mpo_500/xacros/sick_laser.xacro (robot description, xacro)
@@ -4,5 +4,5 @@
     <joint name="${name}_joint" type="fixed">
       <axis xyz="0 1 0" />
-      <insert_block name="origin" />
+      <xacro:insert_block name="origin" />
       <parent link="${parent}"/>
       <child link="${name}_link"/>

File: robot_model/mpo_500/xacros/ultrasonic.xacro (robot description, xacro)
@@ -4,5 +4,5 @@
     <joint name="${name}_joint" type="fixed">
       <axis xyz="0 1 0" />
-      <insert_block name="origin" />
+      <xacro:insert_block name="origin" />
       <parent link="${parent}"/>
       <child link="${name}_link"/>
