Commit message: update robot model to new folder path

File: robot_model/mpo_500.urdf.xacro (robot description, xacro)
@@ -2,16 +2,16 @@
 <robot name="mpo_500" xmlns:xacro="http://www.ros.org/wiki/xacro">
   <!--GAZEBO REFERENCES -->
-  <!-- <xacro:include filename="$(find neo_mpo_500)/robot_model/mpo_500/xacros/mpo_500_gazebo.xacro" /> -->
+  <!-- <xacro:include filename="$(find neo_mpo_500)/robot_model/xacros/mpo_500_gazebo.xacro" /> -->
   <!-- BODY -->
-  <xacro:include filename="$(find neo_mpo_500)/robot_model/mpo_500/xacros/mpo_500_body.xacro" />
+  <xacro:include filename="$(find neo_mpo_500)/robot_model/xacros/mpo_500_body.xacro" />
   <!-- WHEELS -->
-  <xacro:include filename="$(find neo_mpo_500)/robot_model/mpo_500/xacros/omni_wheel.xacro" />
+  <xacro:include filename="$(find neo_mpo_500)/robot_model/xacros/omni_wheel.xacro" />
   <!-- SENSORS -->
   <!-- Sick S300 - Comment/Uncomment if required  -->
-  <xacro:include filename="$(find neo_mpo_500)/robot_model/mpo_500/xacros/sick_S300.xacro" />
+  <xacro:include filename="$(find neo_mpo_500)/robot_model/xacros/sick_S300.xacro" />
   <!-- Microscan - Comment/Uncomment if required -->
-  <!-- <xacro:include filename="$(find neo_mpo_500)/robot_model/mpo_500/xacros/micro_scan.xacro" />
-  <xacro:include filename="$(find neo_mpo_500)/robot_model/mpo_500/xacros/imu.xacro" />
-  <xacro:include filename="$(find neo_mpo_500)/robot_model/mpo_500/xacros/ultrasonic.xacro" />-->
+  <!-- <xacro:include filename="$(find neo_mpo_500)/robot_model/xacros/micro_scan.xacro" />
+  <xacro:include filename="$(find neo_mpo_500)/robot_model/xacros/imu.xacro" />
+  <xacro:include filename="$(find neo_mpo_500)/robot_model/xacros/ultrasonic.xacro" />-->
   <!-- Base Macro-->
   <xacro:mpo_500_base name="base_link">

File: robot_model/xacros/micro_scan.xacro (robot description, xacro)
@@ -17,5 +17,5 @@
     <origin xyz="-0.0 0 -0.06" rpy="1.57 0 0" />
       <geometry>
-        <mesh filename="package://neo_mpo_500/robot_model/mpo_500/meshes/SICK-MICROSCAN3.dae" scale="0.001 0.001 0.001" />
+        <mesh filename="package://neo_mpo_500/robot_model/meshes/SICK-MICROSCAN3.dae" scale="0.001 0.001 0.001" />
       </geometry>
     </visual>
@@ -23,5 +23,5 @@
     <origin xyz="-0.0 0 -0.06" rpy="1.57 0 0" />
         <geometry>
-          <mesh filename="package://neo_mpo_500/robot_model/mpo_500/meshes/SICK-MICROSCAN3.dae" scale="0.001 0.001 0.001" />
+          <mesh filename="package://neo_mpo_500/robot_model/meshes/SICK-MICROSCAN3.dae" scale="0.001 0.001 0.001" />
           </geometry>
         </collision>

File: robot_model/xacros/mpo_500_body.xacro (robot description, xacro)
@@ -13,5 +13,5 @@
         <origin xyz="0. 0. 0" rpy="-1.571 0 1.571" />
         <geometry>
-            <mesh filename="package://neo_mpo_500/robot_model/mpo_500/meshes/MPO-500-BODY.dae" scale="0.001 0.001 0.001"/>
+            <mesh filename="package://neo_mpo_500/robot_model/meshes/MPO-500-BODY.dae" scale="0.001 0.001 0.001"/>
         </geometry>
       </visual>
@@ -20,5 +20,5 @@
         <geometry>
           <!--<box size="0.68 0.41 0.25"/> -->
-           <mesh filename="package://neo_mpo_500/robot_model/mpo_500/meshes/MPO-500-BODY.dae" scale="0.001 0.001 0.001"/>
+           <mesh filename="package://neo_mpo_500/robot_model/meshes/MPO-500-BODY.dae" scale="0.001 0.001 0.001"/>
         </geometry>
       </collision>

File: robot_model/xacros/omni_wheel.xacro (robot description, xacro)
@@ -20,5 +20,5 @@
      <origin xyz="0 0 0" rpy="0 0 0"/>
      <geometry>
-        <mesh filename="package://neo_mpo_500/robot_model/mpo_500/meshes/MPO-500-WHEEL.dae" scale="0.001 0.001 0.001"/>
+        <mesh filename="package://neo_mpo_500/robot_model/meshes/MPO-500-WHEEL.dae" scale="0.001 0.001 0.001"/>
      </geometry>
     </visual>
@@ -26,5 +26,5 @@
      <origin xyz="0 0 0" rpy="0 0 0" />
      <geometry>
-        <mesh filename="package://neo_mpo_500/robot_model/mpo_500/meshes/MPO-500-WHEEL.dae" scale="0.001 0.001 0.001"/>
+        <mesh filename="package://neo_mpo_500/robot_model/meshes/MPO-500-WHEEL.dae" scale="0.001 0.001 0.001"/>
      </geometry>
     </collision>

File: robot_model/xacros/sick_S300.xacro (robot description, xacro)
@@ -17,5 +17,5 @@
         <origin xyz="0 0 -0.12" rpy="-1.57 0 3.14" />
         <geometry>
-        <mesh filename="package://neo_mpo_500/robot_model/mpo_500/meshes/SICK-S300.dae" scale="0.001 0.001 0.001" />
+        <mesh filename="package://neo_mpo_500/robot_model/meshes/SICK-S300.dae" scale="0.001 0.001 0.001" />
         </geometry>
       </visual>
@@ -23,5 +23,5 @@
         <origin xyz="0 0 -0.12" rpy="-1.57 0 3.14" />
         <geometry>
-        <mesh filename="package://neo_mpo_500/robot_model/mpo_500/meshes/SICK-S300.dae" scale="0.001 0.001 0.001" />
+        <mesh filename="package://neo_mpo_500/robot_model/meshes/SICK-S300.dae" scale="0.001 0.001 0.001" />
         </geometry>
       </collision>

File: robot_model/xacros/sick_laser.xacro (robot description, xacro)
@@ -18,5 +18,5 @@
       <origin xyz="0 0 -0.12" rpy="-1.57 0 3.14" />
         <geometry>
-        <mesh filename="package://neo_mpo_500/robot_model/mpo_500/meshes/SICK-S300.dae" scale="0.001 0.001 0.001" />
+        <mesh filename="package://neo_mpo_500/robot_model/meshes/SICK-S300.dae" scale="0.001 0.001 0.001" />
         </geometry>
       </visual>
@@ -24,5 +24,5 @@
         <origin xyz="0 0 0" rpy="-1.57 0 3.14" />
         <geometry>
-        <mesh filename="package://neo_mpo_500/robot_model/mpo_500/meshes/SICK-S300.dae" scale="0.001 0.001 0.001" />
+        <mesh filename="package://neo_mpo_500/robot_model/meshes/SICK-S300.dae" scale="0.001 0.001 0.001" />
         </geometry>
       </collision>
@@ -30,5 +30,5 @@
 <!--  <origin xyz="-0.0 0 -0.06" rpy="1.57 0 0" />
       <geometry>
-      <mesh filename="package://neo_mpo_500/robot_model/mpo_500/meshes/SICK-MICROSCAN3.dae" scale="0.001 0.001 0.001" />
+      <mesh filename="package://neo_mpo_500/robot_model/meshes/SICK-MICROSCAN3.dae" scale="0.001 0.001 0.001" />
       </geometry>
       </visual>
@@ -36,5 +36,5 @@
  <origin xyz="-0.0 0 -0.06" rpy="1.57 0 0" />
       <geometry>
-        <mesh filename="package://neo_mpo_500/robot_model/mp_500/meshes/SICK-MICROSCAN3.dae" scale="0.001 0.001 0.001" />
+        <mesh filename="package://neo_mpo_500/robot_model/meshes/SICK-MICROSCAN3.dae" scale="0.001 0.001 0.001" />
         </geometry>
       </collision> -->

Commit message: update launch files and parameters

File: robot_model/mpo_500.urdf.xacro (robot description, xacro)
@@ -11,7 +11,7 @@
   <xacro:include filename="$(find neo_mpo_500)/robot_model/xacros/sick_S300.xacro" />
   <!-- Microscan - Comment/Uncomment if required -->
-  <!-- <xacro:include filename="$(find neo_mpo_500)/robot_model/xacros/micro_scan.xacro" />
+  <xacro:include filename="$(find neo_mpo_500)/robot_model/xacros/micro_scan.xacro" />
   <xacro:include filename="$(find neo_mpo_500)/robot_model/xacros/imu.xacro" />
-  <xacro:include filename="$(find neo_mpo_500)/robot_model/xacros/ultrasonic.xacro" />-->
+  <xacro:include filename="$(find neo_mpo_500)/robot_model/xacros/ultrasonic.xacro" />
   <!-- Base Macro-->
   <xacro:mpo_500_base name="base_link">
@@ -39,7 +39,7 @@
        <!--+++++++++++++++++++ IMU ++++++++++++++++++++++++-->
  <!-- Comment or uncomment based on your requirement -->
-<!--   <xacro:imu name="imu_1" parent="base_link">
-    <origin xyz="0.100 0 0.300" rpy="0 0 3.14" />
-  </xacro:imu> -->
+  <!--xacro:imu name="imu_1" parent="base_link">
+    <origin xyz="0.100 0 0.300" rpy="0 3.14 3.14" />
+  </xacro:imu-->
   <!--+++++++++++++++++++ Ultra Sonic ++++++++++++++++++++++++-->
   <!-- Comment or uncomment based on your requirement -->

Commit message: mpo_500 updated

File: robot_model/mpo_500.urdf.xacro (robot description, xacro)
@@ -20,23 +20,23 @@
 <!-- Melodic -->
   <!-- Base Macro-->
-<!-- <link name="base_link" /> -->
+<link name="base_link" />
   <!-- Base link macro -->
-<!--   <xacro:mpo_500_base name="base_footprint" parent="base_link">
+  <xacro:mpo_500_base name="base_footprint" parent="base_link">
     <origin xyz="0 0 0" rpy="0 0 0" />
+  </xacro:mpo_500_base>
+<!-- Kinetic -->
+<!--   <xacro:mpo_500_base name="base_link">
   </xacro:mpo_500_base> -->
-<!-- Kinetic -->
-  <xacro:mpo_500_base name="base_link">
-  </xacro:mpo_500_base>
   <!-- Wheel Macro -->
-  <xacro:omni_wheel_250 name="mpo_500_wheel_front_left" parent="base_link">
+  <xacro:omni_wheel_250 name="mpo_500_wheel_front_left" parent="base_footprint">
   	<origin xyz="0.25 0.28 0.13" rpy="0 0 0" />
   </xacro:omni_wheel_250>
-  <xacro:omni_wheel_250 name="mpo_500_wheel_front_right" parent="base_link">
+  <xacro:omni_wheel_250 name="mpo_500_wheel_front_right" parent="base_footprint">
   	<origin xyz="0.25 -0.28 0.13" rpy="0 0 3.14" />
   </xacro:omni_wheel_250>
-  <xacro:omni_wheel_250 name="mpo_500_wheel_back_left" parent="base_link">
+  <xacro:omni_wheel_250 name="mpo_500_wheel_back_left" parent="base_footprint">
   	<origin xyz="-0.25 0.28 0.13" rpy="0 0 0" />
   </xacro:omni_wheel_250>
-  <xacro:omni_wheel_250 name="mpo_500_wheel_back_right" parent="base_link">
+  <xacro:omni_wheel_250 name="mpo_500_wheel_back_right" parent="base_footprint">
   	<origin xyz="-0.25 -0.28 0.13" rpy="0 0 3.14" />
   </xacro:omni_wheel_250>

File: robot_model/urdf/mpo_500_xacros/mpo_500_body.xacro (robot description, xacro)
@@ -1,5 +1,16 @@
 <?xml version="1.0"?>
 <robot name="mmo_500" xmlns:xacro="http://ros.org/wiki/xacro">
-<xacro:macro name="mpo_500_base" params="name">
+<!-- Melodic -->
+ <xacro:macro name="mpo_500_base" params="name parent *origin">
+  <joint name="${name}_joint" type="fixed">
+    <xacro:insert_block name="origin" />
+    <axis xyz="0 0 -1" />
+    <joint_properties damping="1" friction="1" />
+    <parent link="${parent}" />
+    <child link="${name}" />
+   </joint>
+<!-- Kinetic -->
+<!-- <xacro:macro name="mpo_500_base" params="name"> -->
+<!-- Link -->
   <link name="${name}">
     <inertial>

Commit message: No difference between kinetic and melodic

File: robot_model/mpo_500.urdf.xacro (robot description, xacro)
@@ -18,5 +18,4 @@
   <!-- ur5 -->
   <xacro:include filename="$(find neo_mpo_500)/robot_model/urdf/ur_5_xacros/ur5.urdf.xacro" />
-<!-- Melodic -->
   <!-- Base Macro-->
 <link name="base_link" />
@@ -25,7 +24,4 @@
     <origin xyz="0 0 0" rpy="0 0 0" />
   </xacro:mpo_500_base>
-<!-- Kinetic -->
-<!--   <xacro:mpo_500_base name="base_link">
-  </xacro:mpo_500_base> -->
   <!-- Wheel Macro -->
   <xacro:omni_wheel_250 name="mpo_500_wheel_front_left" parent="base_footprint">

File: robot_model/urdf/mpo_500_xacros/mpo_500_body.xacro (robot description, xacro)
@@ -10,6 +10,4 @@
     <child link="${name}" />
    </joint>
-<!-- Kinetic -->
-<!-- <xacro:macro name="mpo_500_base" params="name"> -->
 <!-- Link -->
   <link name="${name}">
